File: hardware/reference/pcb/pcb.kicad_sch (KiCad schematic)
At the start: 63 parts, among them J1 POWER, J2 Conn_01x03, J3 Conn_01x03, J4 Conn_02x03_Odd_Even, J5 485, J6 Conn_01x03, J7 SMA, SW1 SW_Push, U1 AMS1117-3.3, U2 AK09911C, U3 MAX13487EESA, U4 STM32F103C8Tx, U5 DS3231M, U6 NEO-M8M, Y1 8MHz, Y2 32.768kHz

Commit message: Validate config fields
Parts:
- removed C7, C9: 20pF, Capacitor_THT:C_Disc_D3.0mm_W2.0mm_P2.50mm, symbol Device:C_Small
- removed Y2: 32.768kHz, Crystal:Crystal_DS26_D2.0mm_L6.0mm_Horizontal, symbol Device:Crystal_Small
- renumbered C12 to C10, C13 to C11, C14 to C12, C8 to C7, C10 to C8, C11 to C9, R9 to R10, R10 to R8, R8 to R9
Connections:
- net MCU_OSC0: no longer names the net of U4.3 (PC14)
- net MCU_OSC1: no longer names the net of U4.4 (PC15)
- no-connect marks 36 -> 38
Other:
- moved on the sheet: C6, C7, Y1
