File: hardware/gnss/pcb/pcb.kicad_pcb (KiCad board)
At the start: 2 copper layers, 100 x 50 mm, 41 parts, among them J1 POWER, J2 SMA, J3 SMA, J4 RS485, U1 AMS1117-3.3, U2 LC02H, U3 74HC14, U4 MAX3485

Commit message: With QGNSS tool
Parts:
- added D2: SS34, Diode_SMD:D_SMA, F.Cu at (88.5, 84.0)
- moved C1 6.46 mm to (90.0, 92.0)
- renumbered D2 to D3, D3 to D4, D4 to D5, D5 to D6
Routing:
- net /VBAT: track 49.5 -> 57.2 mm
- net /+3V3: track 201.0 -> 205.5 mm
- net /Vin: track 22.8 -> 23.8 mm
