File: hardware/gnss/pcb/pcb.kicad_sch (KiCad schematic)
At the start: 40 parts, among them J1 POWER, J2 SMA, J3 SMA, J4 RS485, U1 AMS1117-3.3, U2 LC02H, U3 74HC14, U4 MAX3485

Commit message: With QGNSS tool
Parts:
- added D2: SS34, Diode_SMD:D_SMA, symbol PCM_Diode_Schottky_AKL:SS34
- renumbered D2 to D3, D3 to D4, D4 to D5, D5 to D6
Connections:
- net +3V3: now also D2.1 (K)
- net VBAT: now also D2.2 (A)
Other:
- moved on the sheet: BT1
