File: hardware/monitor/pcb/pcb.kicad_pcb (KiCad board)
At the start: 2 copper layers, 122 x 122 mm, 50 parts, among them J1 USB_B_Micro, J2 USB_A, J3 USB_A, J4 USB_A, M1 Fan, Q1 S8050, SW1 SW_Push, U1 locked, U2 AT89C52, U3 SL2.1A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

Commit message: Update GNSS schematic
Connections:
- U1 pad 1: unconnected-(U1-A0-Pad1) -> GND
- U1 pad 2: unconnected-(U1-A1-Pad2) -> GND
- U1 pad 3: unconnected-(U1-A2-Pad3) -> GND
Other:
- board text removed: "BUSY"
- board text removed: "ERROR"
- board text removed: "PING"
- board text removed: "POWER"
Changed lines of the file:
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@@
   (net 83 "Net-(D5-A)")
   (net 84 "Net-(D6-A)")
-  (net 85 "unconnected-(U1-A0-Pad1)")
-  (net 86 "unconnected-(U1-A1-Pad2)")
-  (net 87 "unconnected-(U1-A2-Pad3)")
-  (net 88 "/MCU_PING")
+  (net 85 "/MCU_PING")
   (footprint "Connector_USB:USB_A_CONNFLY_DS1095-WNR0" locked (layer "F.Cu")
     (at 171 90 90)
@@
       (net 24 "/MCU_BUSY") (pinfunction "P2.3") (pintype "bidirectional"))
     (pad "25" thru_hole oval locked (at 15.24 38.1) (size 1.6 1.6) (drill 0.8) (layers "*.Cu" "*.Mask")
-      (net 88 "/MCU_PING") (pinfunction "P2.4") (pintype "bidirectional"))
+      (net 85 "/MCU_PING") (pinfunction "P2.4") (pintype "bidirectional"))
     (pad "26" thru_hole oval locked (at 15.24 35.56) (size 1.6 1.6) (drill 0.8) (layers "*.Cu" "*.Mask")
       (net 23 "/MCU_POWER") (pinfunction "P2.5") (pintype "bidirectional"))
@@
       (stroke (width 0.1) (type solid)) (layer "F.Fab"))
     (pad "1" smd roundrect locked (at -4.65 -4.445) (size 2.05 0.6) (layers "F.Cu" "F.Paste" "F.Mask") (roundrect_rratio 0.25)
-      (net 85 "unconnected-(U1-A0-Pad1)") (pinfunction "A0") (pintype "input+no_connect"))
+      (net 2 "GND") (pinfunction "A0") (pintype "input"))
     (pad "2" smd roundrect locked (at -4.65 -3.175) (size 2.05 0.6) (layers "F.Cu" "F.Paste" "F.Mask") (roundrect_rratio 0.25)
-      (net 86 "unconnected-(U1-A1-Pad2)") (pinfunction "A1") (pintype "input+no_connect"))
+      (net 2 "GND") (pinfunction "A1") (pintype "input"))
     (pad "3" smd roundrect locked (at -4.65 -1.905) (size 2.05 0.6) (layers "F.Cu" "F.Paste" "F.Mask") (roundrect_rratio 0.25)
-      (net 87 "unconnected-(U1-A2-Pad3)") (pinfunction "A2") (pintype "input+no_connect"))
+      (net 2 "GND") (pinfunction "A2") (pintype "input"))
     (pad "4" smd roundrect locked (at -4.65 -0.635) (size 2.05 0.6) (layers "F.Cu" "F.Paste" "F.Mask") (roundrect_rratio 0.25)
       (net 27 "/EXP_P0") (pinfunction "P0") (pintype "bidirectional"))
@@
       (net 83 "Net-(D5-A)") (pintype "passive"))
     (pad "2" thru_hole oval locked (at 7.62 0) (size 1.4 1.4) (drill 0.7) (layers "*.Cu" "*.Mask")
-      (net 88 "/MCU_PING") (pintype "passive"))
+      (net 85 "/MCU_PING") (pintype "passive"))
     (model "${KICAD6_3DMODEL_DIR}/Resistor_THT.3dshapes/R_Axial_DIN0204_L3.6mm_D1.6mm_P7.62mm_Horizontal.wrl"
       (offset (xyz 0 0 0))
@@
   (gr_rect locked (start 63 38) (end 185 160)
     (stroke (width 0.15) (type default)) (fill none) (layer "Edge.Cuts"))
-  (gr_text "BUSY" (at 92.7 156.1) (layer "F.SilkS")
+  (gr_text locked "BUSY" (at 92.7 156.1) (layer "F.SilkS")
     (effects (font (size 1.5 1.5) (thickness 0.1875)) (justify bottom))
   )
@@
     (effects (font (size 1.5 1.5) (thickness 0.1875)) (justify bottom))
   )
-  (gr_text "ERROR" (at 100.7 156.1) (layer "F.SilkS")
+  (gr_text locked "ERROR" (at 100.7 156.1) (layer "F.SilkS")
     (effects (font (size 1.5 1.5) (thickness 0.1875)) (justify bottom))
   )
@@
     (effects (font (size 1.5 1.5) (thickness 0.1875)) (justify bottom))
   )
-  (gr_text "PING" (at 100.7 146) (layer "F.SilkS")
+  (gr_text locked "PING" (at 100.7 146) (layer "F.SilkS")
     (effects (font (size 1.5 1.5) (thickness 0.1875)) (justify bottom))
   )
-  (gr_text "POWER" (at 92.6 146) (layer "F.SilkS")
+  (gr_text locked "POWER" (at 92.6 146) (layer "F.SilkS")
     (effects (font (size 1.5 1.5) (thickness 0.1875)) (justify bottom))
   )
@@
   (segment locked (start 179.5375 138) (end 177.310908 138) (width 0.25) (layer "F.Cu") (net 11))
   (segment locked (start 166.970908 142.99) (end 163.193604 142.99) (width 0.25) (layer "F.Cu") (net 13))
-  (segment locked (start 169.24 140.720908) (end 166.970908 142.99) (width 0.25) (layer "F.Cu") (net 13))
   (segment locked (start 160.975 140.771396) (end 160.975 72.525) (width 0.25) (layer "F.Cu") (net 13))
-  (segment locked (start 163.193604 142.99) (end 160.975 140.771396) (width 0.25) (layer "F.Cu") (net 13))
   (segment locked (start 160.975 72.525) (end 171 62.5) (width 0.25) (layer "F.Cu") (net 13))
+  (segment locked (start 169.24 140.720908) (end 166.970908 142.99) (width 0.25) (layer "F.Cu") (net 13))
+  (segment locked (start 163.193604 142.99) (end 160.975 140.771396) (width 0.25) (layer "F.Cu") (net 13))
+  (segment locked (start 170.51 140.34) (end 170.51 141.314999) (width 0.25) (layer "F.Cu") (net 14))
+  (segment locked (start 168.384999 143.44) (end 163.007208 143.44) (width 0.25) (layer "F.Cu") (net 14))
+  (segment locked (start 163.007208 143.44) (end 160.525 140.957792) (width 0.25) (layer "F.Cu") (net 14))
   (segment locked (start 160.525 140.957792) (end 160.525 70.975) (width 0.25) (layer "F.Cu") (net 14))
   (segment locked (start 160.525 70.975) (end 171 60.5) (width 0.25) (layer "F.Cu") (net 14))
   (segment locked (start 170.51 141.314999) (end 168.384999 143.44) (width 0.25) (layer "F.Cu") (net 14))
-  (segment locked (start 168.384999 143.44) (end 163.007208 143.44) (width 0.25) (layer "F.Cu") (net 14))
-  (segment locked (start 170.51 140.34) (end 170.51 141.314999) (width 0.25) (layer "F.Cu") (net 14))
-  (segment locked (start 163.007208 143.44) (end 160.525 140.957792) (width 0.25) (layer "F.Cu") (net 14))
-  (segment locked (start 163.622696 142.09) (end 162.025 140.492304) (width 0.25) (layer "F.Cu") (net 15))
-  (segment locked (start 165.924999 142.09) (end 163.622696 142.09) (width 0.25) (layer "F.Cu") (net 15))
-  (segment locked (start 166.7 141.314999) (end 165.924999 142.09) (width 0.25) (layer "F.Cu") (net 15))
-  (segment locked (start 162.025 140.492304) (end 162.025 128.42) (width 0.25) (layer "F.Cu") (net 15))
-  (segment locked (start 161.875 96.625) (end 171 87.5) (width 0.25) (layer "F.Cu") (net 15))
-  (segment locked (start 166.7 140.34) (end 166.7 141.314999) (width 0.25) (layer "F.Cu") (net 15))
-  (segment locked (start 161.875 128.27) (end 161.875 96.625) (width 0.25) (layer "F.Cu") (net 15))
-  (segment locked (start 162.025 128.42) (end 161.875 128.27) (width 0.25) (layer "F.Cu") (net 15))
-  (segment locked (start 161.575 140.735) (end 161.575 130.16) (width 0.25) (layer "F.Cu") (net 16))
-  (segment locked (start 166.150908 142.54) (end 163.38 142.54) (width 0.25) (layer "F.Cu") (net 16))
-  (segment locked (start 163.38 142.54) (end 161.575 140.735) (width 0.25) (layer "F.Cu") (net 16))
+  (segment locked (start 165.924999 142.09) (end 166.7 141.314999) (width 0.25) (layer "F.Cu") (net 15))
+  (segment locked (start 171 87.5) (end 161.875 96.625) (width 0.25) (layer "F.Cu") (net 15))
+  (segment locked (start 161.875 96.625) (end 161.875 140.342304) (width 0.25) (layer "F.Cu") (net 15))
+  (segment locked (start 161.875 140.342304) (end 163.622696 142.09) (width 0.25) (layer "F.Cu") (net 15))
+  (segment locked (start 163.622696 142.09) (end 165.924999 142.09) (width 0.25) (layer "F.Cu") (net 15))
+  (segment locked (start 166.7 141.314999) (end 166.7 140.34) (width 0.25) (layer "F.Cu") (net 15))
+  (segment locked (start 163.38 142.54) (end 161.425 140.585) (width 0.25) (layer "F.Cu") (net 16))
   (segment locked (start 161.425 95.075) (end 171 85.5) (width 0.25) (layer "F.Cu") (net 16))
-  (segment locked (start 161.575 130.16) (end 161.425 130.01) (width 0.25) (layer "F.Cu") (net 16))
+  (segment locked (start 166.150908 142.54) (end 163.38 142.54) (width 0.25) (layer "F.Cu") (net 16))
   (segment locked (start 167.97 140.720908) (end 166.150908 142.54) (width 0.25) (layer "F.Cu") (net 16))
-  (segment locked (start 161.425 130.01) (end 161.425 95.075) (width 0.25) (layer "F.Cu") (net 16))
+  (segment locked (start 161.425 140.585) (end 161.425 95.075) (width 0.25) (layer "F.Cu") (net 16))
   (segment locked (start 162.925 139.105) (end 162.925 120.575) (width 0.25) (layer "F.Cu") (net 17))
   (segment locked (start 164.16 140.34) (end 162.925 139.105) (width 0.25) (layer "F.Cu") (net 17))
@@
   (segment locked (start 101.775 151.34) (end 99.09 154.025) (width 0.25) (layer "B.Cu") (net 84))
   (segment locked (start 77.025 154.025) (end 76 153) (width 0.25) (layer "B.Cu") (net 84))
-  (segment locked (start 84.645 133.655) (end 84.645 143.975) (width 0.25) (layer "F.Cu") (net 88))
-  (segment locked (start 98.68 119.62) (end 84.645 133.655) (width 0.25) (layer "F.Cu") (net 88))
-  (segment locked (start 84.645 143.975) (end 83.62 145) (width 0.25) (layer "F.Cu") (net 88))
-  (zone (net 2) (net_name "GND") (layers "F&B.Cu") (hatch edge 0.5)
+  (segment locked (start 84.645 133.655) (end 84.645 143.975) (width 0.25) (layer "F.Cu") (net 85))
+  (segment locked (start 98.68 119.62) (end 84.645 133.655) (width 0.25) (layer "F.Cu") (net 85))
+  (segment locked (start 84.645 143.975) (end 83.62 145) (width 0.25) (layer "F.Cu") (net 85))
+  (zone locked (net 2) (net_name "GND") (layers "F&B.Cu") (hatch edge 0.5)
     (connect_pads (clearance 0.3))
     (min_thickness 0.25) (filled_areas_thickness no)
