File: hardware/monitor/pcb/pcb.kicad_sch (KiCad schematic)
At the start: 48 parts, among them J1 USB_B_Micro, J2 USB_A, J3 USB_A, J4 USB_A, M1 Fan, Q1 S8050, SW1 SW_Push, U1 PCF8574, U2 AT89C52, U3 SL2.1A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

Commit message: Update GNSS schematic
Connections:
- net GND: now also U1.1 (A0), U1.2 (A1), U1.3 (A2)
- no-connect marks 43 -> 40
Changed lines of the file:
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@@
   (junction (at 146.685 183.515) (diameter 0) (color 0 0 0 0)
   )
+  (junction (at 210.185 52.705) (diameter 0) (color 0 0 0 0)
+  )
   (junction (at 144.145 183.515) (diameter 0) (color 0 0 0 0)
   )
@@
   (junction (at 128.905 164.465) (diameter 0) (color 0 0 0 0)
   )
+  (junction (at 228.6 71.755) (diameter 0) (color 0 0 0 0)
+  )
   (junction (at 18.415 86.995) (diameter 0) (color 0 0 0 0)
   )
@@
   )
   (junction (at 208.28 42.545) (diameter 0) (color 0 0 0 0)
+  )
+  (junction (at 210.185 55.245) (diameter 0) (color 0 0 0 0)
   )
   (junction (at 111.125 183.515) (diameter 0) (color 0 0 0 0)
@@
   (no_connect (at 245.11 114.3))
   (no_connect (at 130.81 62.865))
-  (no_connect (at 215.9 55.245))
   (no_connect (at 166.37 47.625))
   (no_connect (at 166.37 65.405))
   (no_connect (at 166.37 32.385))
   (no_connect (at 130.81 65.405))
-  (no_connect (at 215.9 52.705))
   (no_connect (at 130.81 75.565))
   (no_connect (at 166.37 56.515))
@@
   (no_connect (at 53.975 153.67))
   (no_connect (at 130.81 37.465))
-  (no_connect (at 215.9 50.165))
   (no_connect (at 166.37 67.945))
   (no_connect (at 130.81 29.845))
@@
     (stroke (width 0) (type default))
   )
+  (wire (pts (xy 210.185 55.245) (xy 210.185 71.755))
+    (stroke (width 0) (type default))
+  )
   (wire (pts (xy 154.305 172.085) (xy 163.195 172.085))
     (stroke (width 0) (type default))
@@
     (stroke (width 0) (type default))
   )
+  (wire (pts (xy 210.185 55.245) (xy 215.9 55.245))
+    (stroke (width 0) (type default))
+  )
   (wire (pts (xy 110.49 34.925) (xy 110.49 38.735))
     (stroke (width 0) (type default))
@@
     (stroke (width 0) (type default))
   )
+  (wire (pts (xy 210.185 52.705) (xy 210.185 55.245))
+    (stroke (width 0) (type default))
+  )
   (wire (pts (xy 22.86 81.915) (xy 18.415 81.915))
     (stroke (width 0) (type default))
@@
     (stroke (width 0) (type default))
   )
+  (wire (pts (xy 210.185 71.755) (xy 228.6 71.755))
+    (stroke (width 0) (type default))
+  )
   (wire (pts (xy 110.49 60.325) (xy 110.49 62.23))
     (stroke (width 0) (type default))
@@
     (stroke (width 0) (type default))
   )
+  (wire (pts (xy 210.185 50.165) (xy 210.185 52.705))
+    (stroke (width 0) (type default))
+  )
   (wire (pts (xy 26.67 41.91) (xy 26.67 44.45))
     (stroke (width 0) (type default))
@@
     (stroke (width 0) (type default))
   )
-  (wire (pts (xy 228.6 70.485) (xy 228.6 74.93))
+  (wire (pts (xy 228.6 70.485) (xy 228.6 71.755))
     (stroke (width 0) (type default))
   )
@@
     (stroke (width 0) (type default))
   )
+  (wire (pts (xy 228.6 71.755) (xy 228.6 74.93))
+    (stroke (width 0) (type default))
+  )
   (wire (pts (xy 110.49 29.845) (xy 110.49 34.925))
     (stroke (width 0) (type default))
@@
     (stroke (width 0) (type default))
   )
+  (wire (pts (xy 215.9 50.165) (xy 210.185 50.165))
+    (stroke (width 0) (type default))
+  )
   (wire (pts (xy 193.04 45.085) (xy 205.74 45.085))
     (stroke (width 0) (type default))
@@
     (stroke (width 0) (type default))
   )
+  (wire (pts (xy 210.185 52.705) (xy 215.9 52.705))
+    (stroke (width 0) (type default))
+  )
