File: drivers/gnss/hardware/pcb/pcb.kicad_pcb (KiCad board)
At the start: 2 copper layers, 100 x 50 mm, 42 parts, among them J1 POWER, J2 SMA, J3 SMA, J4 RS485, U1 AMS1117-3.3, U2 LC02H, U3 74HC14, U4 MAX3485

Commit message: Add LNA schematic & PCB design
Routing:
- net Net-(D1-A): track 15.7 -> 16.7 mm
Other:
- board text added: "2024 全国大学生嵌入式芯片与系统设计竞赛"
- board text added: "GNSS_A"
- board text added: "GNSS_B"
- board text added: "PPS_A"
- board text added: "PPS_B"
- board text added: "RS485_B RS485_A"
- board text added: "RXD"
- board text added: "TXD"
- board text added: "V- V+"
- board text added: "便携式卫星地面站 姿态参考模组"
- board text removed: "locked"

Commit message: Update GNSS PCB
Parts:
- moved D3 0.22 mm to (104.5, 83.8)
- moved D2 0.17 mm to (88.3, 84.0), turned to 0 degrees
Connections:
- D2 pad 1: /+3V3 -> /VBAT
- D2 pad 2: /VBAT -> /+3V3
Routing:
- net /Vin: track 23.8 -> 27.8 mm
